File: rocket_payload/rocket_payload.kicad_pcb (KiCad board)
At the start: 4 copper layers, 73.7 x 73.7 mm, 109 parts, among them J1 Micro_SD_Card, J2 Conn_02x10_Counter_Clockwise, J3 USB_C_Receptacle_USB2.0_14P, J4 Conn_Coaxial_Small, SW1 SW_Push, SW2 SW_Push, U1 STM32H743AIIx, U2 BQ24072RGT, U3 TPS63031DSK, U4 BNO055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

Commit message: added esp
Parts:
- added C60: 100n, Capacitor_SMD:C_0402_1005Metric, F.Cu at (196.1, 132.8)
- added C61: 1u, Capacitor_SMD:C_0402_1005Metric, F.Cu at (196.1, 134.8)
- added C62: 10u, Capacitor_SMD:C_0805_2012Metric, F.Cu at (211.6, 138.0)
- added C63: 100n, Capacitor_SMD:C_0402_1005Metric, F.Cu at (196.1, 136.8)
- added D8: BAT54J, Diode_SMD:D_SOD-323F, F.Cu at (211.5, 141.0)
- added J5: Conn_01x02, Connector_JST:JST_PH_B2B-PH-K_1x02_P2.00mm_Vertical, F.Cu at (155.1, 63.4)
- added J6: USB_C_Receptacle_USB2.0_14P, Connector_USB:USB_C_Receptacle_GCT_USB4085, F.Cu at (157.5, 101.9)
- added R24: 10k, Capacitor_SMD:C_0402_1005Metric, F.Cu at (196.1, 138.7)
- added R25: 10k, Capacitor_SMD:C_0402_1005Metric, F.Cu at (196.1, 140.7)
- added R26: 1M, Resistor_SMD:R_0402_1005Metric, F.Cu at (207.9, 132.8)
- added R27: 5.1k, Resistor_SMD:R_0402_1005Metric, F.Cu at (207.9, 134.8)
- added R28: 5.1k, Resistor_SMD:R_0402_1005Metric, F.Cu at (207.9, 136.8)
- added SW3: SW_Push, Button_Switch_SMD:Panasonic_EVQPUJ_EVQPUA, F.Cu at (202.0, 135.6)
- added U10: ESP32-S3-WROOM-1, RF_Module:ESP32-S3-WROOM-1, F.Cu at (102.6, 92.2)
- added U11: USBLC6-2SC6, Package_TO_SOT_SMD:SOT-23-6, F.Cu at (211.9, 134.2)
- moved C12 117.0 mm to (155.0, 93.8), turned to -90 degrees
- moved C13 115.7 mm to (154.0, 93.8), turned to -90 degrees
- moved C11 114.9 mm to (152.5, 94.0), turned to 90 degrees
- moved SW1 112.9 mm to (100.8, 120.5), turned to 180 degrees
- moved R1 103.0 mm to (100.7, 117.7)
- moved SW2 99.0 mm to (108.7, 120.4), turned to 180 degrees
- moved C4 93.3 mm to (108.6, 117.5), turned to 180 degrees
- moved C30 92.6 mm to (135.0, 85.3)
- moved C31 92.4 mm to (135.0, 86.3)
- moved C34 91.5 mm to (134.0, 88.5), turned to -90 degrees
- moved C35 89.9 mm to (132.9, 88.5), turned to -90 degrees
- moved C36 88.4 mm to (131.8, 88.5), turned to -90 degrees
- moved C37 86.9 mm to (130.7, 88.5), turned to -90 degrees
- moved C38 85.4 mm to (129.6, 88.5), turned to -90 degrees
- moved C40 84.3 mm to (127.4, 88.5), turned to -90 degrees
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Connections:
- U1 pad L9: unconnected-(U1-PB10-PadL9) -> /ESP_RX
- U1 pad M9: unconnected-(U1-PB11-PadM9) -> /ESP_TX
Other:
- board size 73.7 x 73.7 mm -> 70 x 70 mm

Commit message: located all components
Parts:
- added Q1: DMG2301L, Package_TO_SOT_SMD:SOT-23, F.Cu at (105.0, 111.5)
- added R29: 100K, Resistor_SMD:R_0402_1005Metric, F.Cu at (109.5, 113.0)
- added R30: 10k, Resistor_SMD:R_0402_1005Metric, F.Cu at (111.5, 113.0)
- moved R15 136.0 mm to (63.8, 99.3), turned to -90 degrees
- moved C33 118.0 mm to (66.8, 99.3), turned to 180 degrees
- moved C9 118.0 mm to (154.0, 97.0)
- moved C10 117.9 mm to (154.0, 98.5)
- moved SW3 111.9 mm to (98.0, 94.4), turned to 90 degrees
- moved C54 107.8 mm to (157.6, 111.5), turned to 180 degrees
- moved C2 107.2 mm to (139.5, 79.5), turned to -90 degrees
- moved C14 103.3 mm to (134.0, 98.0), turned to -90 degrees
- moved C3 102.3 mm to (140.5, 79.5), turned to -90 degrees
- moved C48 101.3 mm to (157.5, 74.0)
- moved C15 99.4 mm to (135.0, 98.0), turned to -90 degrees
- moved C29 99.2 mm to (141.5, 79.5), turned to -90 degrees
- moved R19 96.5 mm to (104.0, 79.5), turned to 90 degrees
- moved R16 96.4 mm to (109.5, 110.0), turned to 180 degrees
- moved L1 95.4 mm to (116.0, 116.5)
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Connections:
- U1 pad H6: unconnected-(U1-PA4-PadH6) -> /ESP_EN
- U1 pad L4: unconnected-(U1-PA5-PadL4) -> /GPS_SWITCH
Other:
- board text added: "Built by Mason Huslig 2026"
- board text added: "GUPATRON"
