File: rocket_payload/rocket_payload.kicad_pcb (KiCad board)
At the start: 4 copper layers, 70 x 70 mm, 127 parts, among them J1 Micro_SD_Card, J2 Conn_02x10_Counter_Clockwise, J3 USB_C_Receptacle_USB2.0_14P, J4 Conn_Coaxial_Small, J5 Conn_01x02, J6 USB_C_Receptacle_USB2.0_14P, Q1 DMG2301L, SW1 SW_Push, SW2 SW_Push, SW3 SW_Push, U1 STM32H743AIIx, U10 ESP32-S3-WROOM-1, U11 USBLC6-2SC6, U2 BQ24072RGT, U3 TPS63031DSK, U4 BNO055, U5 CH340G, U6 BME280, U7 BMP280, U8 ZOE-M8Q, U9 USBLC6-2SC6, Y1 8MHz Crystal, Y2 12MHz

Commit message: newest board changes
Parts:
- removed J2: Conn_02x10_Counter_Clockwise, Connector_PinSocket_2.00mm:PinSocket_2x10_P2.00mm_Vertical
- added C33: 100nf, Capacitor_SMD:C_0402_1005Metric, B.Cu at (134.0, 110.5)
- added C49: 100nf, Capacitor_SMD:C_0402_1005Metric, B.Cu at (135.2, 110.5)
- added C64: 100n, Capacitor_SMD:C_0402_1005Metric, B.Cu at (142.8, 91.5)
- added C65: 10uf, Capacitor_SMD:C_0402_1005Metric, B.Cu at (135.4, 68.6)
- added C66: 100nf, Capacitor_SMD:C_0402_1005Metric, B.Cu at (135.4, 67.5)
- added C67: 10pf, Capacitor_SMD:C_0402_1005Metric, B.Cu at (140.0, 68.6)
- added C68: 10nf, Capacitor_SMD:C_0402_1005Metric, B.Cu at (132.8, 110.5)
- added C69: 0.1u, Capacitor_SMD:C_0402_1005Metric, B.Cu at (138.2, 111.0)
- added C70: 10u, Capacitor_SMD:C_0402_1005Metric, B.Cu at (139.5, 111.0)
- added C71: 0.1u, Capacitor_SMD:C_0402_1005Metric, B.Cu at (137.0, 111.0)
- added C72: 1u, Capacitor_SMD:C_0402_1005Metric, B.Cu at (156.5, 78.2)
- added J7: Conn_Coaxial_Small, Connector_Coaxial:SMA_Amphenol_132289_EdgeMount, F.Cu at (137.0, 62.6)
- added J8: Conn_01x08_Pin, Connector_JST:JST_EH_S8B-EH_1x08_P2.50mm_Horizontal, F.Cu at (127.0, 107.0)
- added R15: 1M, Resistor_SMD:R_0402_1005Metric, B.Cu at (158.1, 77.6)
- added R31: 1M, Resistor_SMD:R_0402_1005Metric, B.Cu at (158.1, 78.7)
- added REF**: MountingHole_3.2mm_M3, MountingHole:MountingHole_3.2mm_M3, F.Cu at (125.0, 65.0)
- added REF**: MountingHole_3.2mm_M3, MountingHole:MountingHole_3.2mm_M3, F.Cu at (175.0, 115.0)
- added REF**: MountingHole_3.2mm_M3, MountingHole:MountingHole_3.2mm_M3, F.Cu at (125.0, 115.0)
- added U12: BMP581, MyModel:BMP581, F.Cu at (145.0, 91.5)
- added U13: RFM96W-433S2, RFM9X:RFM9X-SMD, B.Cu at (133.4, 78.3)
- added U14: ICM-42688-P, ICM42688:PQFN50P300X250X97-14N, F.Cu at (132.0, 108.0)
- added U15: LSM6DSV16XTR, LSM6DSV:XDCR_LSM6DSV16XTR, F.Cu at (138.0, 108.0)
- C1, C10, C11, C12, C13, C14, C15, C16, C17, C18, C19, C2, C20, C21, C22, C23, C24, C25, C26, C27, C28, C29, C3, C30, C31, C32, C33, C34, C35, C36, C37, C38, C39, C4, C40, C41, C42, C43, C44, C45, C46, C47, C48, C49, C5, C50, C51, C52, C53, C54, C55, C56, C57, C58, C59, C6, C60, C61, C62, C63, C7, C8, C9, D1, D7, D8, FB1, J1, L1, L2, Q1, R1, R10, R11, R12, R13, R14, R15, R16, R17, R18, R19, R2, R20, R21, R22, R23, R24, R25, R26, R27, R28, R29, R3, R30, R4, R5, R6, R7, R8, R9, U11, U2, U3, U5, U9, Y1, Y2: moved to B.Cu
- J4: footprint Connector_Coaxial:U.FL_Hirose_U.FL-R-SMT-1_Vertical -> Connector_Coaxial:SMA_Amphenol_132289_EdgeMount
- J5: footprint Connector_JST:JST_PH_B2B-PH-K_1x02_P2.00mm_Vertical -> Connector_JST:JST_EH_S2B-EH_1x02_P2.50mm_Horizontal
- U1: footprint Package_BGA:UFBGA-169_7x7mm_Layout13x13_P0.5mm -> Package_QFP:LQFP-100_14x14mm_P0.5mm
- moved J4 86.5 mm to (165.0, 62.6), turned to 90 degrees
- moved C23 85.3 mm to (167.0, 67.2)
- moved D7 85.3 mm to (174.3, 70.1)
- moved SW3 83.6 mm to (178.4, 71.4), turned to -90 degrees
- moved R15 78.3 mm to (141.4, 89.1)
- moved Q1 78.0 mm to (173.8, 74.9), turned to 180 degrees
- moved U8 77.0 mm to (170.0, 70.0), turned to 0 degrees
- moved C49 76.2 mm to (142.6, 89.1), turned to 90 degrees
- moved R30 75.3 mm to (175.0, 72.5), turned to 180 degrees
- moved R29 74.8 mm to (170.7, 70.0), turned to -90 degrees
- moved C33 72.8 mm to (138.8, 89.2)
- moved R16 71.0 mm to (170.7, 74.1), turned to -90 degrees
- moved L1 69.5 mm to (169.5, 72.1), turned to -90 degrees
- moved C50 68.8 mm to (168.4, 70.0), turned to -90 degrees
- moved C25 68.3 mm to (165.6, 72.1), turned to 0 degrees
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Connections:
- net Net-(D2-DOUT) renamed /DIN1
- net Net-(D3-DOUT) renamed /DIN2
Routing:
- net /USB_VDD: track 0.00 -> 61.6 mm, vias 0 -> 3
- net +3.3V: track 0.00 -> 33.4 mm, vias 0 -> 4
- net /ESP_D_plus_usb: track 0.00 -> 19.5 mm
- net Net-(D1-A): track 0.00 -> 17.9 mm
- net /DIN1: track 0.00 -> 16.2 mm, vias 0 -> 2
- net Net-(D8-A): track 0.00 -> 16.2 mm
- net /ESP_D_minus_usb: track 0.00 -> 15.5 mm
- net Net-(J6-CC2): track 0.00 -> 13.9 mm
- net Net-(J3-CC2): track 0.00 -> 11.1 mm
- net /BOOT: track 0.00 -> 10.3 mm, vias 0 -> 1
- net /DIN2: track 0.00 -> 9.68 mm, vias 0 -> 2
- net /GPS_SWITCH: track 0.00 -> 9.32 mm
- net /RF_IN: track 0.00 -> 8.77 mm, vias 0 -> 3
- net Net-(J7-In): track 0.00 -> 8.41 mm, vias 0 -> 1
- net /RESET: track 0.00 -> 7.57 mm, vias 0 -> 1
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- added copper zone on In2.Cu, net +3.3V
- added copper zone on In1.Cu, net GND
Other:
- board size 70 x 70 mm -> 60 x 60 mm
- board text added: "D12"
- board text added: "D13"
- board text added: "D14"
- board text added: "D15"
- board text added: "E0"
- board text added: "E1"
- board text added: "E2"
- board text added: "ESP"
- board text added: "Gupatron v1.0"
- board text added: "STM"
- board text removed: "Built by Mason Huslig 2026"
- board text removed: "GUPATRON"

Commit message: lots of routing
Parts:
- removed C34, C35, C36, C42, C43, C44, C45: 100n, Capacitor_SMD:C_0402_1005Metric
- removed C55, C56, C57: 2.2u, Capacitor_SMD:C_0402_1005Metric
- removed U1: STM32H743AIIx, Package_QFP:LQFP-100_14x14mm_P0.5mm
- added U16: STM32H7A3VGTx, Package_QFP:LQFP-100_14x14mm_P0.5mm, F.Cu at (150.0, 77.5)
- moved C29 10.2 mm to (143.0, 84.7), turned to 0 degrees
- moved U9 10.2 mm to (169.5, 78.1)
- moved C41 9.90 mm to (162.0, 78.0), turned to 0 degrees
- moved C3 9.61 mm to (143.0, 85.8), turned to 0 degrees
- moved C2 9.26 mm to (143.0, 86.9), turned to 180 degrees
- moved C40 9.11 mm to (162.0, 76.9), turned to 0 degrees
- moved U2 8.78 mm to (167.8, 106.1), turned to 0 degrees
- moved C72 8.67 mm to (149.2, 73.5)
- moved R31 8.67 mm to (150.8, 74.0)
- moved R15 8.67 mm to (150.8, 72.9)
- moved C39 8.40 mm to (162.0, 75.8), turned to 0 degrees
- moved C31 8.15 mm to (149.9, 70.4), turned to 45 degrees
- moved C38 7.97 mm to (162.0, 74.7), turned to 0 degrees
- moved FB1 7.91 mm to (146.6, 88.7)
- moved C37 6.49 mm to (162.0, 79.1), turned to 0 degrees
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Routing:
- net /STM_SCL: track 0.00 -> 79.5 mm, vias 0 -> 15
- net /PD12: track 0.00 -> 59.7 mm, vias 0 -> 3
- net /SCL_3V: track 0.00 -> 58.0 mm, vias 0 -> 6
- net /SDMMC_D2: track 1.73 -> 59.5 mm, vias 0 -> 9
- net /PD13: track 0.00 -> 53.8 mm, vias 0 -> 4
- net /SDA_3V: track 0.00 -> 52.8 mm, vias 0 -> 7
- net /PD15: track 0.00 -> 52.7 mm, vias 0 -> 4
- net /PD14: track 0.00 -> 50.6 mm, vias 0 -> 5
- net /LSM_INT: track 0.00 -> 48.7 mm, vias 0 -> 4
- net /ICP_CS: track 0.00 -> 45.7 mm, vias 0 -> 4
- net /STM_MISO: track 0.30 -> 40.6 mm, vias 0 -> 3
- net /SDMMC_D1: track 1.69 -> 40.8 mm, vias 0 -> 4
- net /SDMMC_D0: track 1.69 -> 37.3 mm, vias 0 -> 5
- net /PE0: track 0.00 -> 35.3 mm, vias 0 -> 2
- net /USB_VDD: track 61.6 -> 93.2 mm, vias 3 -> 7
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Other:
- board text added: "Made by: Mason Huslig"

Commit message: added new traces
Parts:
- moved C22 1.66 mm to (143.5, 76.0)
- moved C58 1.60 mm to (145.6, 75.3), turned to 180 degrees
- moved C30 1.40 mm to (158.2, 77.1)
- moved C54 0.50 mm to (153.0, 89.3)
- moved C40 0.44 mm to (162.2, 76.5)
- moved C37 0.44 mm to (162.2, 78.7)
- moved C38 0.44 mm to (162.2, 74.3)
- moved C39 0.44 mm to (162.2, 75.4)
- moved C41 0.44 mm to (162.2, 77.5)
- moved R10 0.27 mm to (135.4, 105.5)
- moved C16 0.25 mm to (134.2, 105.5)
- moved R21 0.16 mm to (136.8, 105.6)
- moved C20 0.14 mm to (154.6, 91.7)
- moved C19 0.14 mm to (154.6, 88.1)
Routing:
- net /LSM_CS: track 0.00 -> 101.3 mm, vias 0 -> 11
- net /ESP_RX: track 0.00 -> 44.6 mm, vias 0 -> 5
- net /GPS_SWITCH: track 9.32 -> 51.8 mm, vias 0 -> 3
- net /ICP42688_INT: track 21.4 -> 62.9 mm, vias 2 -> 3
- net /SDMMC_D3: track 1.69 -> 42.5 mm, vias 0 -> 5
- net /Interrupt21: track 1.58 -> 40.8 mm, vias 1 -> 7
- net /STM_MOSI: track 26.3 -> 60.6 mm, vias 2 -> 8
- net /STM_GPS_TIME: track 0.00 -> 31.7 mm, vias 0 -> 4
- net /STM_RESET_PIN: track 0.00 -> 28.3 mm, vias 0 -> 6
- net /LORA_RESET: track 7.13 -> 29.3 mm, vias 1 -> 5
- net /ESP_TX: track 28.4 -> 48.6 mm, vias 3 -> 6
- net /SDMMC_CMD: track 1.69 -> 17.1 mm, vias 0 -> 5
- net /SCL_3V: track 58.0 -> 70.8 mm, vias 6 -> 11
- net /LORA_NSS: track 27.7 -> 40.0 mm, vias 5 -> 4
- net /LORA_DIO0: track 0.14 -> 12.0 mm, vias 0 -> 2
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