File: rocket_payload/rocket_payload.kicad_sch (KiCad schematic)
At the start: 49 parts, among them J1 Micro_SD_Card, J2 Conn_Coaxial_Small, P1 USB_C_Plug_USB2.0, Q1 FDN340P, U1 ATmega2560-16C, U2 LM358, U3 LP2985-3.3, U4 BNO055, U5 CH340G, U6 BME280, U7 BMP280, U8 ZOE-M8Q, U9 RFM96W-433S2, Y1 16Mhz, Y2 12MHz

Commit message: added changes
Parts:
- removed P1: USB_C_Plug_USB2.0, symbol Connector:USB_C_Plug_USB2.0
- removed R2: 27R, symbol Device:R
- removed R5: 10k, symbol Device:R
- removed U1: ATmega2560-16C, Package_BGA:TFBGA-100_9.0x9.0mm_Layout10x10_P0.8mm, symbol MCU_Microchip_ATmega:ATmega2560-16C
- removed Y1: 16Mhz, symbol Device:Crystal_GND2
- added C22, C23, C26, C27, C28, C29, C33, C34, C35, C36, C37, C38, C39, C40, C41, C42, C43, C44, C45: 100n, symbol Device:C
- added C24: 0.1u, symbol Device:C
- added C25: 4.7u, symbol Device:C
- added C30, C31: 0.2u, symbol Device:C
- added C32: 1u, symbol Device:C
- added D2, D3, D4: SK6812, LED_SMD:LED_SK6812_PLCC4_5.0x5.0mm_P3.2mm, symbol LED:SK6812
- added J3: USB_C_Receptacle_USB2.0_14P, symbol Connector:USB_C_Receptacle_USB2.0_14P
- added L1: 2.2u, symbol Device:L
- added Q2, Q3: BSS138, Package_TO_SOT_SMD:SOT-23, symbol Transistor_FET:BSS138
- added R13, R14, R15, R16: 4.7k, symbol Device:R
- added R17: 1k, symbol Device:R
- added R18: 5.1k, symbol Device:R
- added U1: STM32H743AIIx, Package_BGA:UFBGA-169_7x7mm_Layout13x13_P0.5mm, symbol MCU_ST_STM32H7:STM32H743AIIx
- added U10: TXS0108EPW, Package_SO:TSSOP-20_4.4x6.5mm_P0.65mm, symbol Logic_LevelTranslator:TXS0108EPW
- C1, C3: value 100n -> 1u
- C4: value 22p -> 100n
- R1: value 1M -> 10k
Connections:
- net +3.3V: now also U8.D4 (D_SEL), U8.H9 (V_BCKP), U8.J1 (VCC), U8.J2 (VCC), C23.1, C24.1, C32.1, C33.1, Q2.2 (S), Q3.2 (S), R13.1, R16.1, U1.C4 (PDR_ON), U1.G12 (VDD50_USB), U1.G13 (VDD33_USB), U10.10 (OE), U10.2 (VCCA)
- net +5V: now also C22.1, C26.1, C27.1, C28.1, D2.3 (VDD), D3.3 (VDD), D4.3 (VDD), R14.1, R15.1, U10.19 (VCCB); no longer C1.1, C2.1
- net GND: now also R1.1, U8.A1 (GND), U8.A3 (GND), U8.A5 (GND), U8.A7 (GND), U8.A8 (GND), U8.A9 (GND), U8.B9 (GND), U8.C7 (GND), U8.C9 (GND), U8.D6 (GND), U8.D9 (GND), U8.E7 (GND), U8.F7 (GND), U8.G3 (GND), U8.G6 (GND), U8.G7 (GND), U8.J3 (GND), U8.J9 (GND), C22.2, C23.2, C24.2, C25.1, C26.2, C27.2, C28.2, C29.2, C30.1, C31.1, C32.2, C33.2, C34.2, C35.2, C36.2, C37.2, C38.2, C39.2, C40.2, C41.2, C42.2, C43.2, C44.2, C45.2, D2.1 (VSS), D3.1 (VSS), D4.1 (VSS), R18.2, U1.B10 (VSS), U1.B3 (VSS), U1.C12 (VSS), U1.D2 (VSS), U1.G2 (VSS), U1.H12 (VSS), U1.J3 (VSSA), U1.L12 (VSS), U1.M11 (VSS), U1.M2 (VSS), U1.M4 (VSS), U1.M7 (VSS), U10.11 (GND)
- net RadioInterrupt: now also R17.2; no longer U9.14 (DIO0)
- net Reset: no longer C4.1
- net SCL: no longer J1.5 (CLK), R3.2, U4.20 (COM0), U7.4 (SCK), U9.4 (SCK)
- net SDA: no longer R4.2, U4.19 (COM1), U7.3 (SDI)
- net XTAL1: now also U1.H1 (PH0); no longer R1.2
- net XTAL2: now also U1.H2 (PH1); no longer R1.1
- net at U5.5 (UD+): now also J3.A6 (D+), J3.B6 (D+)
- net at U5.6 (UD-): now also J3.A7 (D-), J3.B7 (D-)
- net at R9.1: now also J3.A5 (CC1)
- net SDA_3V: now reaches U8.A2 (SDA/~{SPI_CS})
- net SDA_3V: now also U4.19 (COM1), U7.3 (SDI), Q2.1 (G), R13.2
- net Antenna: now reaches U8.A4 (RF_IN)
- net SCL_3V: now reaches U8.B1 (SCL/SPI_CLK)
- net SCL_3V: now also U4.20 (COM0), U7.4 (SCK), U9.4 (SCK), Q3.1 (G), R16.2
- net at U8.G1 (V_CORE): now also C25.2, L1.1
- net at U8.H1 (V_DCDC_OUT): now also L1.2
- net ZOE_RX_3V: now reaches U8.J4 (RXD/SPI_MOSI)
- net ZOE_RX_3V: now also U10.8 (A7)
- net ZOE_TX_3V: now reaches U8.J5 (TXD/SPI_MISO)
- net ZOE_TX_3V: now also U10.7 (A6)
- net VREF: now reaches C3.1
- net VREF: now also C29.1, U1.L2 (VREF+)
- net at C8.1, R8.1: now also J3.A1 (GND), J3.A12 (GND), J3.B1 (GND), J3.B12 (GND)
- net at C8.2, R8.2: now also J3.S1 (SHIELD)
- net ANTENNA: now reaches J2.1 (In), U9.9 (ANT)
- net at D1.2 (A): now also J3.A4 (VBUS), J3.A9 (VBUS), J3.B4 (VBUS), J3.B9 (VBUS)
- net CS renamed SD_CS_3V
- net MISO renamed MISO_3V
- net MISO_3V: now also U10.18 (B2)
- net MOSI renamed MOSI_3V
- net MOSI_3V: now also U10.20 (B1)
- net RadioCS renamed CS_LORA_3V
- net CS_LORA_3V: now also U10.16 (B4)
- new net: J3.B5 (CC2), R18.1
- new net: C30.2, C31.2, U1.D13 (VCAP), U1.N10 (VCAP)
- new net: D3.4 (DOUT), D4.2 (DIN)
- new net: D2.4 (DOUT), D3.2 (DIN)
- new net: R17.1, U9.14 (DIO0)
- new net: R1.2, U1.E6 (BOOT0)
- new net CS_LORA_5V: U10.5 (A4)
- new net CS_ZOE_3V: U10.15 (B5)
- new net CS_ZOE_5V: U10.6 (A5)
- new net LED_PIN: D2.2 (DIN)
- new net MISO_5V: U10.3 (A2)
- new net MOSI_5V: U10.1 (A1)
- new net RESET: C4.1, U1.G6 (NRST)
- new net SCK_3V: J1.5 (CLK), U10.17 (B3)
- new net SCK_5V: U10.4 (A3)
- new net SCL_5V: Q3.3 (D), R15.2, R3.2
- new net SDA_5V: Q2.3 (D), R14.2, R4.2
- new net VBAT: U1.E3 (VBAT)
- new net VDDA: C1.1, C2.1, U1.L1 (VDDA)
- new net VDD_MCU: C34.1, C35.1, C36.1, C37.1, C38.1, C39.1, C40.1, C41.1, C42.1, C43.1, C44.1, C45.1, U1.A10 (VDD), U1.A3 (VDD), U1.A7 (VDD), U1.B4 (VDDLDO), U1.C13 (VDD), U1.D1 (VDD), U1.D12 (VDDLDO), U1.G1 (VDD), U1.H13 (VDD), U1.L13 (VDD), U1.M1 (VDD), U1.M10 (VDDLDO), U1.N11 (VDD), U1.N4 (VDD), U1.N7 (VDD)
- new net ZOE_RX_5V: U10.13 (B7)
- new net ZOE_TX_5V: U10.14 (B6)
- no-connect marks 15 -> 27
Other:
- note added: "Comm Level Shifting"
- note added: "I2C Level Shifting"
- note added: "NEOPIXEL_LED"
- note removed: "*need to change I2C logic level"
- moved on the sheet: C12, C13, C14, C15, C16, C8, D1, R10, R8, R9, U4, Y2

Commit message: finished schematic
Parts:
- removed J2: Conn_Coaxial_Small, symbol Connector:Conn_Coaxial_Small
- removed Q1: FDN340P, Package_TO_SOT_SMD:SOT-23, symbol Transistor_FET:FDN340P
- removed Q2, Q3: BSS138, Package_TO_SOT_SMD:SOT-23, symbol Transistor_FET:BSS138
- removed U2: LM358, symbol Amplifier_Operational:LM358
- removed U3: LP2985-3.3, Package_TO_SOT_SMD:SOT-23-5, symbol Regulator_Linear:LP2985-3.3
- removed U9: RFM96W-433S2, symbol RF_Module:RFM96W-433S2
- added C46, C47: 10u, symbol Device:C
- added C48: 0.3u, symbol Device:C
- added C49, C50, C52, C53, C54: 100n, symbol Device:C
- added C51: 47u, symbol Device:C
- added C55, C56, C57: 2.2u, symbol Device:C
- added D5, D6: LED, symbol Device:LED
- added FB1: FerriteBead, symbol Device:FerriteBead
- added J2: Conn_02x10_Counter_Clockwise, symbol Connector_Generic:Conn_02x10_Counter_Clockwise
- added L2: 1.5u, symbol Device:L
- added R19, R20, R21, R5: 10k, symbol Device:R
- added R2: 1.18k, symbol Device:R
- added SW1, SW2: SW_Push, symbol Switch:SW_Push
- added U2: BQ24072RGT, Package_DFN_QFN:VQFN-16-1EP_3x3mm_P0.5mm_EP1.6x1.6mm, symbol Battery_Management:BQ24072RGT
- added U3: TPS63031DSK, Package_SON:WSON-10-1EP_2.5x2.5mm_P0.5mm_EP1.2x2mm, symbol Regulator_Switching:TPS63031DSK
- added U9: USBLC6-2SC6, Package_TO_SOT_SMD:SOT-23-6, symbol Power_Protection:USBLC6-2SC6
- C21, C33, C6: value 100n -> 10u
- C32: value 1u -> 47u
- C5, C7: value 100n -> 4.7u
- R15, R16: value 4.7k -> 10k
- R17: value 1k -> 10k
- R3: value 10k -> 1.13k
- R7: value 10k -> 330
Connections:
- net RadioInterrupt is gone; now on net SDMMC_D2: R17.2
- net SCL is gone; now on net SCL_3V: U6.4 (SCK)
- net SDA is gone; now on net SDA_3V: U6.3 (SDI)
- net SD_CS_3V is gone; now on net SDMMC_D3: J1.2 (DAT3/CD)
- net VREF is gone; now on net VDDA: C29.1, C3.1, U1.L2 (VREF+)
- net +3.3V: now also R11.1, R14.1, R15.2, R17.1, C46.1, C49.1, C50.1, C51.1, C52.1, C53.1, C54.1, FB1.1, J2.1 (Pin_1), J2.20 (Pin_20), R19.1, R20.1, R21.1, SW1.1, U3.1 (VOUT), U3.10 (FB); no longer C32.1, R11.2, U1.C4 (PDR_ON)
- net CH340G_RX: now also U1.E11 (PA9)
- net CH340G_TX: now also U1.E10 (PA10)
- net GND: now also C5.2, C6.2, R1.2, R3.2, R4.1, U8.C4 (~{SAFEBOOT}), U8.J7 (RTC_I), C46.2, C47.2, C48.2, C49.2, C50.2, C51.2, C52.2, C53.2, C54.2, C55.2, C56.2, C57.2, J2.10 (Pin_10), J2.9 (Pin_9), R2.2, SW2.2, U2.15 (TD), U2.17 (VSS), U2.4 (~{CE}), U2.5 (EN2), U2.8 (VSS), U3.11 (PGND), U3.3 (PGND), U3.9 (GND), U9.2 (GND); no longer R1.1
- net Interrupt21: now also U1.M5 (PB0), R21.2
- net LED_PIN: now also R7.1; no longer D2.2 (DIN)
- net MISO_3V: no longer J1.7 (DAT0)
- net MOSI_3V: no longer J1.3 (CMD)
- net RESET: now also SW2.1
- net SCK_3V: no longer J1.5 (CLK)
- net SCL_3V: now also R13.2, U1.A5 (PB6), U4.19 (COM1); no longer R16.2, U4.20 (COM0)
- net SDA_3V: now also R14.2, U1.D6 (PB7), U4.20 (COM0); no longer R13.2, U4.19 (COM1)
- net VDDA: now also FB1.2
- net VDD_MCU: no longer U1.B4 (VDDLDO), U1.D12 (VDDLDO), U1.M10 (VDDLDO)
- net ZOE_RX_3V: no longer U8.J4 (RXD/SPI_MOSI)
- net ZOE_TX_3V: no longer U8.J5 (TXD/SPI_MISO)
- net D_plus_usb: now reaches J3.A6 (D+), J3.B6 (D+)
- net D_plus_usb: now also U9.3 (I/O2); no longer U5.5 (UD+)
- net D_minus_usb: now reaches J3.A7 (D-), J3.B7 (D-)
- net D_minus_usb: now also U9.1 (I/O1); no longer U5.6 (UD-)
- net SDMMC_D1: now reaches R12.2
- net SDMMC_D1: now also J1.8 (DAT1), U1.F11 (PC9); no longer J1.1 (DAT2)
- net at R7.2: now also D2.2 (DIN); no longer C5.2
- net STM_GPS_TIME: now reaches U8.C3 (TIMEPULSE)
- net STM_RESET_PIN: now reaches U8.J6 (~{RESET})
- net STM_RESET_PIN: now also R16.2
- net BOOT: now reaches U1.E6 (BOOT0)
- net BOOT: now also R1.1, SW1.2; no longer R1.2
- net SDMMC_CLK: now reaches U1.A11 (PC12)
- net SDMMC_CLK: now also J1.5 (CLK)
- net SDMMC_D2: now reaches U1.A12 (PC10)
- net SDMMC_D2: now also J1.1 (DAT2)
- net SDMMC_D3: now reaches U1.B11 (PC11)
- net SDMMC_D3: now also R19.2
- net SDMMC_CMD: now reaches U1.E9 (PD2)
- net SDMMC_CMD: now also J1.3 (CMD), R20.2
- net SDMMC_D0: now reaches U1.F12 (PC8)
- net SDMMC_D0: now also J1.7 (DAT0), R11.2
- net Radio_TX: now reaches U1.N1 (PA2)
- net Radio_TX: now also J2.2 (Pin_2)
- net Radio_RX: now reaches U1.N3 (PA3)
- net Radio_RX: now also J2.3 (Pin_3)
- net +3V3 renamed USB_VDD
- net USB_VDD: now also C22.1, C26.1, C27.1, C28.1, C32.1, C9.1, D1.1 (K), D2.3 (VDD), D3.3 (VDD), D4.3 (VDD), R6.2, U10.19 (VCCB), U5.16 (VCC), R5.2, U2.13 (IN), U9.5 (VBUS)
- removed net +5V: C22.1, C26.1, C27.1, C28.1, C7.1, C9.1, D1.1 (K), D2.3 (VDD), D3.3 (VDD), D4.3 (VDD), R14.1, R15.1, R3.1, R4.1, U10.19 (VCCB), U5.16 (VCC)
- removed net CMP: C5.1, R6.2, R7.1
- removed net SCL_5V: R15.2, R3.2
- net SDA_5V: no longer names the net of R4.2
- net SDA_5V: now also U2.1 (TS); no longer R14.2
- net VIN: no longer names the net of R6.1
- net VIN: now also D6.2 (A)
- new net: R3.1, U2.16 (ISET)
- new net: R2.1, U2.12 (ILIM)
- new net: C48.1, U3.6 (EN), U3.7 (PS/SYNC), U3.8 (VINA)
- new net: L2.1, U3.4 (L1)
- new net: L2.2, U3.2 (L2)
- new net: J2.5 (Pin_5), R15.1
- new net: D5.2 (A), R5.1
- new net BAT_POS: C7.1, U2.2 (BAT), U2.3 (BAT)
- new net CHG: D5.1 (K), U2.9 (~{CHG})
- new net D_minus_ch340: U5.6 (UD-), U9.6 (I/O1)
- new net D_plus_ch340: U5.5 (UD+), U9.4 (I/O2)
- new net PDR: U1.C4 (PDR_ON)
- new net PGOOD: D6.1 (K), U2.7 (~{PGOOD})
- new net VDD_LDO_1: C55.1, U1.B4 (VDDLDO)
- new net VDD_LDO_2: C56.1, U1.D12 (VDDLDO)
- new net VDD_LDO_3: C57.1, U1.M10 (VDDLDO)
- new net VSYS: C47.1, C5.1, U2.10 (OUT), U2.11 (OUT), U2.6 (EN1), U3.5 (VIN)
- no-connect marks 27 -> 40
Other:
- note added: "Boot Circuitry"
- note added: "Digi XbeePros3B Socket"
- note added: "ESD Protection"
- note added: "Power Stuff"
- note removed: "I2C Level Shifting"
- note removed: "Power Management"
- note removed: "Radio Module 433"
- moved on the sheet: C1, C2, C24, C25, C26, C29, C3, C4, L1, U8

Commit message: did erc and now schematic is fin
Parts:
- removed U10: TXS0108EPW, Package_SO:TSSOP-20_4.4x6.5mm_P0.65mm, symbol Logic_LevelTranslator:TXS0108EPW
- added C58, C59: 22p, symbol Device:C
- added D7: PRTR5V0U2X, Package_TO_SOT_SMD:SOT-143, symbol Power_Protection:PRTR5V0U2X
- added J4: Conn_Coaxial_Small, symbol Connector:Conn_Coaxial_Small
- added R22, R23: 1k, symbol Device:R
- added Y1: 8MHz Crystal, symbol Device:Crystal
- C23: value 100n -> 10p
Connections:
- net PDR is gone; now on net +3.3V: U1.C4 (PDR_ON)
- net Reset is gone; now on net RESET: C11.2
- net VBAT is gone; now on net +3.3V: U1.E3 (VBAT)
- net VDD_MCU is gone; now on net +3.3V: C34.1, C35.1, C36.1, C37.1, C38.1, C39.1, C40.1, C41.1, C42.1, C43.1, C44.1, C45.1, U1.A10 (VDD), U1.A3 (VDD), U1.A7 (VDD), U1.C13 (VDD), U1.D1 (VDD), U1.G1 (VDD), U1.H13 (VDD), U1.L13 (VDD), U1.M1 (VDD), U1.N11 (VDD), U1.N4 (VDD), U1.N7 (VDD)
- net +3.3V: now also C22.1, D7.4 (VCC), R22.1; no longer C23.1, U6.5 (SDO)
- net GND: now also C58.2, C59.2, D7.1 (GND), J4.2 (Ext), R23.1; no longer C23.2, U7.5 (SDO)
- net LED_PIN: now also U1.E12 (PA8)
- net STM_GPS_TIME: now also U1.L5 (PB1)
- net STM_RESET_PIN: now also U1.L6 (PB2)
- net USB_VDD: no longer C22.1
- net XTAL1: now also C58.1, Y1.1
- net XTAL2: now also C59.1, Y1.2
- net at C30.2, U1.D13 (VCAP): no longer C31.2, U1.N10 (VCAP)
- net Antenna renamed RF_IN
- net RF_IN: now also C23.2, D7.2 (I/O1)
- new net: C31.2, U1.N10 (VCAP)
- new net: R22.2, U6.5 (SDO)
- new net: R23.2, U7.5 (SDO)
- new net: C23.1, J4.1 (In)
- no-connect marks 40 -> 152
Other:
- note added: "MCU POWER"
- note removed: "Comm Level Shifting"
- moved on the sheet: C1, C2, C29, C3, C34, C35, C36, C37, C38, C39, C40, C41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

Commit message: added footprints
Parts:
- C1, C17, C18, C19, C20, C21, C25, C33, C46, C47, C5, C6, C7: footprint (none) -> Capacitor_SMD:C_0805_2012Metric
- C10, C11, C12, C13, C14, C15, C16, C2, C22, C23, C24, C26, C27, C28, C29, C3, C30, C31, C34, C35, C36, C37, C38, C39, C4, C40, C41, C42, C43, C44, C45, C48, C49, C50, C52, C53, C54, C55, C56, C57, C58, C59, C8, C9: footprint (none) -> Capacitor_SMD:C_0402_1005Metric
- C32, C51: footprint (none) -> Capacitor_SMD:C_1206_3216Metric
- D5, D6: footprint (none) -> LED_SMD:LED_0402_1005Metric
- FB1, R1, R10, R11, R12, R13, R14, R15, R16, R17, R18, R19, R2, R20, R21, R22, R23, R3, R4, R5, R6, R7, R8, R9: footprint (none) -> Resistor_SMD:R_0402_1005Metric
- J1: footprint (none) -> Connector_Card:microSD_HC_Hirose_DM3AT-SF-PEJM5
- J2: footprint (none) -> Connector_PinSocket_2.00mm:PinSocket_2x10_P2.00mm_Vertical
- J3: footprint (none) -> Connector_USB:USB_C_Receptacle_GCT_USB4085
- J4: footprint (none) -> Connector_Coaxial:U.FL_Hirose_U.FL-R-SMT-1_Vertical
- L1, L2: footprint (none) -> Inductor_SMD:L_0402_1005Metric
- SW1, SW2: footprint (none) -> Button_Switch_SMD:Panasonic_EVQPUJ_EVQPUA
- Y1, Y2: footprint (none) -> Crystal:Crystal_SMD_3225-4Pin_3.2x2.5mm

Commit message: added esp
Parts:
- added C60, C63: 100n, Capacitor_SMD:C_0402_1005Metric, symbol Device:C
- added C61: 1u, Capacitor_SMD:C_0402_1005Metric, symbol Device:C
- added C62: 10u, Capacitor_SMD:C_0805_2012Metric, symbol Device:C
- added D8: BAT54J, Diode_SMD:D_SOD-323F, symbol Diode:BAT54J
- added J5: Conn_01x02, Connector_JST:JST_PH_B2B-PH-K_1x02_P2.00mm_Vertical, symbol Connector_Generic:Conn_01x02
- added J6: USB_C_Receptacle_USB2.0_14P, Connector_USB:USB_C_Receptacle_GCT_USB4085, symbol Connector:USB_C_Receptacle_USB2.0_14P
- added R24, R25: 10k, Capacitor_SMD:C_0402_1005Metric, symbol Device:R
- added R26: 1M, Resistor_SMD:R_0402_1005Metric, symbol Device:R
- added R27, R28: 5.1k, Resistor_SMD:R_0402_1005Metric, symbol Device:R
- added SW3: SW_Push, Button_Switch_SMD:Panasonic_EVQPUJ_EVQPUA, symbol Switch:SW_Push
- added U10: ESP32-S3-WROOM-1, RF_Module:ESP32-S3-WROOM-1, symbol RF_Module:ESP32-S3-WROOM-1
- added U11: USBLC6-2SC6, Package_TO_SOT_SMD:SOT-23-6, symbol Power_Protection:USBLC6-2SC6
Connections:
- net +3.3V: now also C60.1, C62.1, R24.1, R25.1, U10.2 (3V3)
- net BAT_POS: now also J5.1 (Pin_1)
- net GND: now also C60.2, C61.2, C62.2, J5.2 (Pin_2), R27.2, R28.2, SW3.1, U10.1 (GND), U10.40 (GND), U10.41 (GND), U11.2 (GND)
- net USB_VDD: now also D8.1 (K), U11.5 (VBUS)
- net ESP_RX: now reaches U1.L9 (PB10)
- net ESP_RX: now also U10.36 (RXD0)
- net ESP_TX: now reaches U1.M9 (PB11)
- net ESP_TX: now also U10.37 (TXD0)
- new net: C63.1, J6.A1 (GND), J6.A12 (GND), J6.B1 (GND), J6.B12 (GND), R26.1
- new net: C63.2, J6.S1 (SHIELD), R26.2
- new net: D8.2 (A), J6.A4 (VBUS), J6.A9 (VBUS), J6.B4 (VBUS), J6.B9 (VBUS)
- new net: J6.A5 (CC1), R27.1
- new net: J6.B5 (CC2), R28.1
- new net: R25.2, U10.27 (IO0)
- new net ESP_D+: U10.14 (USB_D+), U11.4 (I/O2)
- new net ESP_D-: U10.13 (USB_D-), U11.6 (I/O1)
- new net ESP_D_minus_usb: J6.A7 (D-), J6.B7 (D-), U11.1 (I/O1)
- new net ESP_D_plus_usb: J6.A6 (D+), J6.B6 (D+), U11.3 (I/O2)
- new net ESP_EN: C61.1, R24.2, SW3.2, U10.3 (EN)
- no-connect marks 152 -> 181
Other:
- note added: "ESP32-S3-WROOM"
- note added: "USB Interface(ESP)"
- note added: "USB Interface(STM)"
- note removed: "USB Interface"

Commit message: located all components
Parts:
- added Q1: DMG2301L, Package_TO_SOT_SMD:SOT-23, symbol Transistor_FET:DMG2301L
- added R29: 100K, Resistor_SMD:R_0402_1005Metric, symbol Device:R
- added R30: 10k, Resistor_SMD:R_0402_1005Metric, symbol Device:R
Connections:
- net +3.3V: now also Q1.2 (S), Q1.3 (D), R30.1
- net ESP_EN: now also U1.H6 (PA4)
- net GND: now also R29.2
- net GPS_SWITCH: now reaches U1.L4 (PA5)
- net GPS_SWITCH: now also Q1.1 (G), R29.1, R30.2
- no-connect marks 181 -> 179
