File: rocket_payload/rocket_payload.kicad_sch (KiCad schematic)
At the start: 127 parts, among them J1 Micro_SD_Card, J2 Conn_02x10_Counter_Clockwise, J3 USB_C_Receptacle_USB2.0_14P, J4 Conn_Coaxial_Small, J5 Conn_01x02, J6 USB_C_Receptacle_USB2.0_14P, Q1 DMG2301L, SW1 SW_Push, SW2 SW_Push, SW3 SW_Push, U1 STM32H743AIIx, U10 ESP32-S3-WROOM-1, U11 USBLC6-2SC6, U2 BQ24072RGT, U3 TPS63031DSK, U4 BNO055, U5 CH340G, U6 BME280, U7 BMP280, U8 ZOE-M8Q, U9 USBLC6-2SC6, Y1 8MHz Crystal, Y2 12MHz

Commit message: newest board changes
Parts:
- removed J2: Conn_02x10_Counter_Clockwise, Connector_PinSocket_2.00mm:PinSocket_2x10_P2.00mm_Vertical, symbol Connector_Generic:Conn_02x10_Counter_Clockwise
- added C64: 100n, Capacitor_SMD:C_0402_1005Metric, symbol Device:C
- added C65: 10uf, Capacitor_SMD:C_0402_1005Metric, symbol Device:C
- added C66: 100nf, Capacitor_SMD:C_0402_1005Metric, symbol Device:C
- added C67: 10pf, Capacitor_SMD:C_0402_1005Metric, symbol Device:C
- added C68: 10nf, Capacitor_SMD:C_0402_1005Metric, symbol Device:C
- added C69, C71: 0.1u, Capacitor_SMD:C_0402_1005Metric, symbol Device:C
- added C70: 10u, Capacitor_SMD:C_0402_1005Metric, symbol Device:C
- added C72: 1u, Capacitor_SMD:C_0402_1005Metric, symbol Device:C
- added J7: Conn_Coaxial_Small, Connector_Coaxial:SMA_Amphenol_132289_EdgeMount, symbol Connector:Conn_Coaxial_Small
- added J8: Conn_01x08_Pin, Connector_JST:JST_EH_S8B-EH_1x08_P2.50mm_Horizontal, symbol Connector:Conn_01x08_Pin
- added R31: 1M, Resistor_SMD:R_0402_1005Metric, symbol Device:R
- added U12: BMP581, MyModel:BMP581, symbol BMP581:BMP581
- added U13: RFM96W-433S2, RFM9X:RFM9X-SMD, symbol RF_Module:RFM96W-433S2
- added U14: ICM-42688-P, ICM42688:PQFN50P300X250X97-14N, symbol ICM-42688-P:ICM-42688-P
- added U15: LSM6DSV16XTR, LSM6DSV:XDCR_LSM6DSV16XTR, symbol LSM6DSV16XTR:LSM6DSV16XTR
- C33: value 10u -> 100nf; footprint Capacitor_SMD:C_0805_2012Metric -> Capacitor_SMD:C_0402_1005Metric
- C49: value 100n -> 100nf
- J4: footprint Connector_Coaxial:U.FL_Hirose_U.FL-R-SMT-1_Vertical -> Connector_Coaxial:SMA_Amphenol_132289_EdgeMount
- J5: footprint Connector_JST:JST_PH_B2B-PH-K_1x02_P2.00mm_Vertical -> Connector_JST:JST_EH_S2B-EH_1x02_P2.50mm_Horizontal
- R15: value 10k -> 1M
- U1: footprint Package_BGA:UFBGA-169_7x7mm_Layout13x13_P0.5mm -> Package_QFP:LQFP-100_14x14mm_P0.5mm
Connections:
- net +3.3V: now also C65.1, C66.1, C69.1, C70.1, U13.13 (3.3V), U15.8 (VDD); no longer C33.1, C49.1, R15.2
- net BAT_POS: now also R15.1
- net GND: now also C64.2, C65.2, C66.2, C68.2, C69.2, C70.2, C71.2, C72.2, J7.2 (Ext), J8.1 (Pin_1), R31.2, U12.3 (GND), U12.8 (GND), U12.9 (GND), U13.1 (GND), U13.10 (GND), U13.8 (GND), U14.11 (RESV_11), U14.6 (GND), U14.7 (RESV_7), U14.9 (INT2/FSYNC/CLKIN), U15.6 (GND), U15.7 (GND)
- net DIN2: now reaches D3.4 (DOUT), D4.2 (DIN)
- net DIN1: now reaches D2.4 (DOUT), D3.2 (DIN)
- net PE2: now reaches U1.A2 (PE2)
- net PE2: now also J8.8 (Pin_8)
- net PE1: now reaches U1.D4 (PE1)
- net PE1: now also J8.7 (Pin_7)
- net PE0: now reaches U1.D5 (PE0)
- net PE0: now also J8.6 (Pin_6)
- net STM_MOSI: now reaches U1.E5 (PF3)
- net STM_MOSI: now also U12.4 (SDI/SDA), U13.3 (MOSI), U14.1 (AP_SDO/AP_AD0), U15.14 (SDA)
- net STM_SCL: now reaches U1.F4 (PF2)
- net STM_SCL: now also U12.2 (SCK/SCL), U13.4 (SCK), U14.13 (AP_SCL/AP_SCLK), U15.13 (SCL)
- net ICP_CS: now reaches U1.F5 (PF5)
- net ICP_CS: now also U14.12 (AP_CS)
- net STM_MISO: now reaches U1.G3 (PF4)
- net STM_MISO: now also U12.5 (SDO/ADR), U13.2 (MISO), U14.14 (AP_SDA/AP_SDIO/AP_SDI), U15.1 (SDO/SA0)
- net LSM_CS: now reaches U1.G4 (PF6)
- net LSM_CS: now also U15.12 (CS)
- net BMP581_CS: now reaches U1.G5 (PF9)
- net BMP581_CS: now also U12.6 (CSB)
- net LORA_FHSS: now reaches U1.G8 (PE7)
- net LORA_FHSS: now also U13.16 (DIO2)
- net BMP581_INT: now reaches U1.H3 (PF10)
- net BMP581_INT: now also U12.7 (INT)
- net LORA_NSS: now reaches U1.H4 (PF8)
- net LORA_NSS: now also U13.5 (NSS)
- net LORA_DIO1: now reaches U1.H8 (PE8)
- net LORA_DIO1: now also U13.15 (DIO1)
- net VOLTAGE_READ: now reaches U1.J1 (PC0)
- net VOLTAGE_READ: now also R15.2, C72.1, R31.1
- net PD13: now reaches U1.J11 (PD13)
- net PD13: now also J8.3 (Pin_3)
- net PD15: now reaches U1.J12 (PD15)
- net PD15: now also J8.5 (Pin_5)
- net PD14: now reaches U1.J13 (PD14)
- net PD14: now also J8.4 (Pin_4)
- net LORA_DIO0: now reaches U1.J8 (PE9)
- net LORA_DIO0: now also U13.14 (DIO0)
- net PD12: now reaches U1.K13 (PD12)
- net PD12: now also J8.2 (Pin_2)
- net ICP42688_INT: now reaches U1.M6 (PF11)
- net ICP42688_INT: now also U14.4 (INT1/INT)
- net LORA_RESET: now reaches U1.M8 (PE10)
- net LORA_RESET: now also U13.6 (RESET)
- net LSM_INT: now reaches U1.N6 (PF12)
- net LSM_INT: now also U15.4 (INT1)
- net Radio_RX: no longer names the net of U1.N3 (PA3)
- net Radio_TX: no longer names the net of U1.N1 (PA2)
- new net: C67.1, U13.9 (ANT)
- new net: C33.1, C49.1, U14.8 (VDD)
- new net: C71.1, U15.5 (VDD_IO)
- new net: C64.1, U12.1 (VDDIO), U12.10 (VDD)
- new net: C67.2, J7.1 (In)
- new net: C68.1, U14.5 (VDDIO)
- no-connect marks 179 -> 157
Other:
- note added: "BMP581 Pressure Sensor"
- note added: "Charging Circuit"
- note added: "Connector"
- note added: "ICP 42688 IMU"
- note added: "IMU Wiring (BNO 055)"
- note added: "Lora Radio"
- note added: "STM IMU"
- note added: "Voltage Reader"
- note removed: "Digi XbeePros3B Socket"
- note removed: "IMU Wiring"
- moved on the sheet: C14, C15, C16, L2, R10, R21, U4

Commit message: lots of routing
Parts:
- removed C34, C35, C36, C42, C43, C44, C45: 100n, Capacitor_SMD:C_0402_1005Metric, symbol Device:C
- removed C55, C56, C57: 2.2u, Capacitor_SMD:C_0402_1005Metric, symbol Device:C
- removed U1: STM32H743AIIx, Package_QFP:LQFP-100_14x14mm_P0.5mm, symbol MCU_ST_STM32H7:STM32H743AIIx
- added U16: STM32H7A3VGTx, Package_QFP:LQFP-100_14x14mm_P0.5mm, symbol MCU_ST_STM32H7:STM32H7A3VGTx
Connections:
- net +3.3V: now also U16.100 (VDD), U16.11 (VDD), U16.27 (VDD), U16.50 (VDD), U16.6 (VBAT), U16.75 (VDD)
- net BMP581_CS: now also U16.85 (PD4)
- net BMP581_INT: now also U16.86 (PD5)
- net BOOT: now also U16.94 (BOOT0)
- net CH340G_RX: now also U16.68 (PA9)
- net CH340G_TX: now also U16.69 (PA10)
- net ESP_EN: now also U16.28 (PA4)
- net ESP_RX: now also U16.46 (PB10)
- net ESP_TX: now also U16.47 (PB11)
- net GND: now also U16.10 (VSS), U16.19 (VSSA), U16.26 (VSS), U16.49 (VSS), U16.74 (VSS), U16.99 (VSS)
- net GPS_SWITCH: now also U16.29 (PA5)
- net ICP42688_INT: now also U16.87 (PD6)
- net ICP_CS: now also U16.41 (PE11)
- net Interrupt21: now also U16.34 (PB0)
- net LED_PIN: now also U16.67 (PA8)
- net LORA_DIO0: now also U16.39 (PE9)
- net LORA_DIO1: now also U16.38 (PE8)
- net LORA_FHSS: now also U16.37 (PE7)
- net LORA_NSS: now also U16.84 (PD3)
- net LORA_RESET: now also U16.40 (PE10)
- net LSM_CS: now also U16.45 (PE15)
- net LSM_INT: now also U16.88 (PD7)
- net PD12: now also U16.59 (PD12)
- net PD13: now also U16.60 (PD13)
- net PD14: now also U16.61 (PD14)
- net PD15: now also U16.62 (PD15)
- net PE0: now also U16.97 (PE0)
- net PE1: now also U16.98 (PE1)
- net PE2: now also U16.1 (PE2)
- net RESET: now also U16.14 (NRST)
- net SCL_3V: now also U16.92 (PB6)
- net SDA_3V: now also U16.93 (PB7)
- net SDMMC_CLK: now also U16.80 (PC12)
- net SDMMC_CMD: now also U16.83 (PD2)
- net SDMMC_D0: now also U16.65 (PC8)
- net SDMMC_D1: now also U16.66 (PC9)
- net SDMMC_D2: now also U16.78 (PC10)
- net SDMMC_D3: now also U16.79 (PC11)
- net STM_GPS_TIME: now also U16.35 (PB1)
- net STM_MISO: now also U16.43 (PE13)
- net STM_MOSI: now also U16.44 (PE14)
- net STM_RESET_PIN: now also U16.36 (PB2)
- net STM_SCL: now also U16.42 (PE12)
- net VDDA: now also U16.20 (VREF+), U16.21 (VDDA)
- net VOLTAGE_READ: now also U16.15 (PC0)
- net XTAL1: now also U16.12 (PH0)
- net XTAL2: now also U16.13 (PH1)
- net at C30.2: now also U16.48 (VCAP)
- net at C31.2: now also U16.73 (VCAP)
- no-connect marks 157 -> 107
Other:
- moved on the sheet: C58, C59, Y1
